File: docs/hardware/kicad/i2c_io.kicad_sch (KiCad schematic)
At the start: 7 parts, among them U22 ADS1115 0x48, U23 ADS1115 0x49, U24 PCF8574 0x20, U26 MPU-6050 0x68, U28 PCA9685 0x40

Commit message: Match the firmware to schematic v0.3: current scaling, contactor checks, fans
- Current sense divides by half the per-pin IS resistor (IS_PIN_RESISTOR_OHMS),
  since R_IS and L_IS are joined; it read about half the real current before.
  The DRIVER level now comes from the resistor (1.8 V with 1k boards).
- DRIVER and OVERCUR open the contactor: a shorted MOSFET ignores DRIVE_EN.
  The drive enable drops before the contactor opens.
- Motor-bus sense: R5-R7 in the schematic (150k/12k to ADS1115 #2 A2, 2.2k
  bleed). New ContactorCheck: K1 stays open at boot until the bus drains
  (K1_WELD if it doesn't, permanent), and NO_BUS when K1 is held closed with
  no bus.
- I2C at 100 kHz, the PCF8574's rating.
- Box fans full on through PCA9685 channel 1; DS18B20 read with our own
  1-Wire timing; new HOT fault (65 C, hysteresis to 55 C).
- WHEEL_REVERSED per wheel in config.h.

Co-Authored-By: Claude Opus 5.5 (1M context) <noreply@anthropic.com>
Claude-Session: https://claude.ai/code/session_01BrgYX7MqpwRKNfNAgoiyH8
Parts:
- U23: Note Steering current sense; A1-A3 spare (A1 reserved for AS5600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 -> Steering current sense (A0), motor bus (A2); A1 reserved fo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
Connections:
- net BUS_SENSE: now reaches U23.A2
- no-connect marks 27 -> 26
Other:
- moved on the sheet: R25, R26, U24, U26, U28
