File: docs/hardware/kicad/controller.kicad_sch (KiCad schematic)
At the start: 14 parts, among them U20 ESP32-WROOM-32D, U21 AION RX Mini, U31 DS18B20

Commit message: Add the listen-only Bluetooth log module
An HC-06 module (U33) hears TX0, the USB serial log, through a 1k
resistor (R29); its TXD is not connected, so nothing on a phone can reach
the ESP32, whose own Wi-Fi and Bluetooth stay off. An Android phone reads
the live log with a serial terminal app.

The phone can't type, so holding the horn for 3 s with the car Locked or
Killed and stopped prints a full report: status, fault table, crash copy
and the last 50 records. `report` on the console does the same. The
trigger is in rideon_core with tests, under SR-31, plus a mutant.

New bt_setup bench firmware sets the module to 115200 baud and a PIN
before it goes in the box. Schematic, wire list, BOM, overview and the 3D
view are regenerated; BLUETOOTH.md, PINOUT, WIRING, SAFETY, README and a
phase 3 commissioning gate describe it.

Co-Authored-By: Claude Opus 5.5 <noreply@anthropic.com>
Parts:
- added R29: 1k, symbol Device:R
- added U33: HC-06, symbol rideonesp32:HC06_BT_Serial
Connections:
- net 5V_LOGIC: now also U33.VCC
- net GND: now also U33.GND
- net LOG_TX: now reaches U20.R3 (TX0/GPIO1)
- net LOG_TX: now also R29.1
- new net BT_RXD: R29.2, U33.RXD
Other:
- note added: "Bluetooth log, listen-only"
Changed lines of the file:
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@@
 (wire (pts (xy 76.2 43.18) (xy 81.28 43.18)) (stroke (width 0) (type default)))
 (global_label "I2C_SCL" (shape passive) (at 81.28 43.18 0) (fields_autoplaced yes) (effects (font (size 1.27 1.27)) (justify left)) (property "Intersheetrefs" "${INTERSHEET_REFS}" (at 81.28 43.18 0) (effects (font (size 1.27 1.27)) (hide yes))))
-(no_connect (at 76.2 45.72))
+(wire (pts (xy 76.2 45.72) (xy 81.28 45.72)) (stroke (width 0) (type default)))
+(label "LOG_TX" (at 81.28 45.72 0) (effects (font (size 1.27 1.27)) (justify left bottom)))
 (no_connect (at 76.2 48.26))
 (wire (pts (xy 76.2 50.8) (xy 81.28 50.8)) (stroke (width 0) (type default)))
@@
 (wire (pts (xy 186.69 132.08) (xy 191.77 132.08)) (stroke (width 0) (type default)))
 (global_label "DF_RX" (shape passive) (at 191.77 132.08 0) (fields_autoplaced yes) (effects (font (size 1.27 1.27)) (justify left)) (property "Intersheetrefs" "${INTERSHEET_REFS}" (at 191.77 132.08 0) (effects (font (size 1.27 1.27)) (hide yes))))
+(text "Bluetooth log, listen-only" (exclude_from_sim no) (at 229.86 27.2 0) (effects (font (size 2 2) (bold yes)) (justify left top)))
+(symbol (lib_id "Device:R") (at 246.38 38.1 90) (unit 1)
+  (exclude_from_sim no) (in_bom yes) (on_board yes) (dnp no)
+  (property "Reference" "R29" (at 246.38 35.284 270) (effects (font (size 1.27 1.27))))
+  (property "Value" "1k" (at 246.38 41.116 270) (effects (font (size 1.27 1.27))))
+  (property "Footprint" "" (at 246.38 38.1 270) (effects (font (size 1.27 1.27)) (hide yes)))
+  (property "Datasheet" "" (at 246.38 38.1 270) (effects (font (size 1.27 1.27)) (hide yes)))
+  (property "Description" "Resistor 1k, metal film 1 %, 0.25 W" (at 246.38 38.1 270) (effects (font (size 1.27 1.27)) (hide yes)))
+  (property "Part" "Resistor 1k, metal film 1 %, 0.25 W" (at 246.38 38.1 270) (effects (font (size 1.27 1.27)) (hide yes)))
+  (property "Source" "Ordered 24 Oct" (at 246.38 38.1 270) (effects (font (size 1.27 1.27)) (hide yes)))
+  (property "Location" "A1" (at 246.38 38.1 270) (effects (font (size 1.27 1.27)) (hide yes)))
+  (property "Note" "Bluetooth RXD series resistor: a dead module can't hold down the USB serial line" (at 246.38 38.1 270) (effects (font (size 1.27 1.27)) (hide yes)))
+  (pin "1")
+  (pin "2")
+  (instances (project "rideonesp32" (path "/e0e78d72-bf5c-51da-8e0f-d8642949b63b/60fb54a3-8b44-551e-9b8a-2c73288ddd08" (reference "R29") (unit 1))))
+)
+(wire (pts (xy 242.57 38.1) (xy 237.49 38.1)) (stroke (width 0) (type default)))
+(label "LOG_TX" (at 237.49 38.1 180) (effects (font (size 1.27 1.27)) (justify right bottom)))
+(wire (pts (xy 250.19 38.1) (xy 255.27 38.1)) (stroke (width 0) (type default)))
+(label "BT_RXD" (at 255.27 38.1 0) (effects (font (size 1.27 1.27)) (justify left bottom)))
+(symbol (lib_id "rideonesp32:HC06_BT_Serial") (at 259.08 53.34 0) (unit 1)
+  (exclude_from_sim no) (in_bom yes) (on_board yes) (dnp no)
+  (property "Reference" "U33" (at 259.08 49 0) (effects (font (size 1.27 1.27))))
+  (property "Value" "HC-06" (at 259.08 60.42 0) (effects (font (size 1.27 1.27))))
+  (property "Footprint" "" (at 259.08 53.34 0) (effects (font (size 1.27 1.27)) (hide yes)))
+  (property "Datasheet" "" (at 259.08 53.34 0) (effects (font (size 1.27 1.27)) (hide yes)))
+  (property "Description" "HC-06 Bluetooth serial module" (at 259.08 53.34 0) (effects (font (size 1.27 1.27)) (hide yes)))
+  (property "Part" "HC-06 Bluetooth serial module" (at 259.08 53.34 0) (effects (font (size 1.27 1.27)) (hide yes)))
+  (property "Source" "To buy" (at 259.08 53.34 0) (effects (font (size 1.27 1.27)) (hide yes)))
+  (property "Location" "box" (at 259.08 53.34 0) (effects (font (size 1.27 1.27)) (hide yes)))
+  (property "Note" "Listen-only log to a phone: hears TX0 (the USB serial log). TXD stays unconnected, so nothing can reach the ESP32. Set to 115200 with the bt_setup bench firmware first" (at 259.08 53.34 0) (effects (font (size 1.27 1.27)) (hide yes)))
+  (pin "VCC")
+  (pin "GND")
+  (pin "RXD")
+  (pin "TXD")
+  (instances (project "rideonesp32" (path "/e0e78d72-bf5c-51da-8e0f-d8642949b63b/60fb54a3-8b44-551e-9b8a-2c73288ddd08" (reference "U33") (unit 1))))
+)
+(wire (pts (xy 248.92 53.34) (xy 243.84 53.34)) (stroke (width 0) (type default)))
+(global_label "5V_LOGIC" (shape passive) (at 243.84 53.34 180) (fields_autoplaced yes) (effects (font (size 1.27 1.27)) (justify right)) (property "Intersheetrefs" "${INTERSHEET_REFS}" (at 243.84 53.34 0) (effects (font (size 1.27 1.27)) (hide yes))))
+(wire (pts (xy 248.92 55.88) (xy 243.84 55.88)) (stroke (width 0) (type default)))
+(global_label "GND" (shape passive) (at 243.84 55.88 180) (fields_autoplaced yes) (effects (font (size 1.27 1.27)) (justify right)) (property "Intersheetrefs" "${INTERSHEET_REFS}" (at 243.84 55.88 0) (effects (font (size 1.27 1.27)) (hide yes))))
+(wire (pts (xy 269.24 53.34) (xy 274.32 53.34)) (stroke (width 0) (type default)))
+(label "BT_RXD" (at 274.32 53.34 0) (effects (font (size 1.27 1.27)) (justify left bottom)))
+(no_connect (at 269.24 55.88))
 (text "Pin nets come from include/pins.h; CI keeps pins.h, PINOUT.md and WIRING.md in step and check_netlist.py checks this sheet." (exclude_from_sim no) (at 15 15 0) (effects (font (size 1.5 1.5) (italic yes)) (justify left top)))
 (text "Analog inputs on ADC1 only. GPIO36/39 carry analog only (they glitch when the ADC runs). Kill lines on pins quiet at boot." (exclude_from_sim no) (at 15 17.6 0) (effects (font (size 1.5 1.5) (italic yes)) (justify left top)))

Commit message: Switch the Bluetooth log module to BLE (HM-10) for iPhone and Android
The HC-06 is Bluetooth Classic, which iPhones can't use. The HM-10 (CC2541)
is BLE, which both iPhone and Android support. Same wiring: RXD on TX0
through R29, TXD not connected.

bt_setup now speaks the HM-10 dialect (genuine and the common clones):
finds the baud rate, names it RideOn, sets 115200, restarts it and checks.
No PIN: HM-10 pairing PINs are unreliable on iPhones and clones, and the
log holds no personal data.

A BLE link passes on about 2 KB/s, so the horn-triggered report prints one
line per 100 ms. A typed report on USB stays at full speed.

Co-Authored-By: Claude Opus 5.5 <noreply@anthropic.com>
Parts:
- U33: value HC-06 -> HM-10; symbol rideonesp32:HC06_BT_Serial -> rideonesp32:HM10_BLE_Serial; Part HC-06 Bluetooth serial module -> HM-10 BLE serial module (iPhone and Android)
Connections:
- no-connect marks 4 -> 6
Changed lines of the file:
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@@
 (wire (pts (xy 250.19 38.1) (xy 255.27 38.1)) (stroke (width 0) (type default)))
 (label "BT_RXD" (at 255.27 38.1 0) (effects (font (size 1.27 1.27)) (justify left bottom)))
-(symbol (lib_id "rideonesp32:HC06_BT_Serial") (at 259.08 53.34 0) (unit 1)
+(symbol (lib_id "rideonesp32:HM10_BLE_Serial") (at 259.08 55.88 0) (unit 1)
   (exclude_from_sim no) (in_bom yes) (on_board yes) (dnp no)
   (property "Reference" "U33" (at 259.08 49 0) (effects (font (size 1.27 1.27))))
-  (property "Value" "HC-06" (at 259.08 60.42 0) (effects (font (size 1.27 1.27))))
-  (property "Footprint" "" (at 259.08 53.34 0) (effects (font (size 1.27 1.27)) (hide yes)))
-  (property "Datasheet" "" (at 259.08 53.34 0) (effects (font (size 1.27 1.27)) (hide yes)))
-  (property "Description" "HC-06 Bluetooth serial module" (at 259.08 53.34 0) (effects (font (size 1.27 1.27)) (hide yes)))
-  (property "Part" "HC-06 Bluetooth serial module" (at 259.08 53.34 0) (effects (font (size 1.27 1.27)) (hide yes)))
-  (property "Source" "To buy" (at 259.08 53.34 0) (effects (font (size 1.27 1.27)) (hide yes)))
-  (property "Location" "box" (at 259.08 53.34 0) (effects (font (size 1.27 1.27)) (hide yes)))
-  (property "Note" "Listen-only log to a phone: hears TX0 (the USB serial log). TXD stays unconnected, so nothing can reach the ESP32. Set to 115200 with the bt_setup bench firmware first" (at 259.08 53.34 0) (effects (font (size 1.27 1.27)) (hide yes)))
+  (property "Value" "HM-10" (at 259.08 62.96 0) (effects (font (size 1.27 1.27))))
+  (property "Footprint" "" (at 259.08 55.88 0) (effects (font (size 1.27 1.27)) (hide yes)))
+  (property "Datasheet" "" (at 259.08 55.88 0) (effects (font (size 1.27 1.27)) (hide yes)))
+  (property "Description" "HM-10 BLE serial module (iPhone and Android)" (at 259.08 55.88 0) (effects (font (size 1.27 1.27)) (hide yes)))
+  (property "Part" "HM-10 BLE serial module (iPhone and Android)" (at 259.08 55.88 0) (effects (font (size 1.27 1.27)) (hide yes)))
+  (property "Source" "To buy" (at 259.08 55.88 0) (effects (font (size 1.27 1.27)) (hide yes)))
+  (property "Location" "box" (at 259.08 55.88 0) (effects (font (size 1.27 1.27)) (hide yes)))
+  (property "Note" "Listen-only log to a phone: hears TX0 (the USB serial log). TXD stays unconnected, so nothing can reach the ESP32. Set to 115200 with the bt_setup bench firmware first" (at 259.08 55.88 0) (effects (font (size 1.27 1.27)) (hide yes)))
   (pin "VCC")
   (pin "GND")
+  (pin "BRK")
   (pin "RXD")
   (pin "TXD")
+  (pin "STATE")
   (instances (project "rideonesp32" (path "/e0e78d72-bf5c-51da-8e0f-d8642949b63b/60fb54a3-8b44-551e-9b8a-2c73288ddd08" (reference "U33") (unit 1))))
 )
@@
 (label "BT_RXD" (at 274.32 53.34 0) (effects (font (size 1.27 1.27)) (justify left bottom)))
 (no_connect (at 269.24 55.88))
+(no_connect (at 269.24 58.42))
+(no_connect (at 248.92 58.42))
 (text "Pin nets come from include/pins.h; CI keeps pins.h, PINOUT.md and WIRING.md in step and check_netlist.py checks this sheet." (exclude_from_sim no) (at 15 15 0) (effects (font (size 1.5 1.5) (italic yes)) (justify left top)))
 (text "Analog inputs on ADC1 only. GPIO36/39 carry analog only (they glitch when the ADC runs). Kill lines on pins quiet at boot." (exclude_from_sim no) (at 15 17.6 0) (effects (font (size 1.5 1.5) (italic yes)) (justify left top)))
