File: docs/hardware/kicad/drive.kicad_sch (KiCad schematic)
At the start: 30 parts, among them U10 IBT-2 FL, U11 IBT-2 FR, U12 IBT-2 RL, U13 IBT-2 RR, U14 IBT-2 STEER

Commit message: Safety gates follow the toy standards; add per-motor fuses F11-F14
SAFETY.md and COMMISSIONING.md now split their checks into required
(what a lab tests on every shop-bought ride-on: EN 71-1 / SI 562-1,
EN 62115, ASTM F963) and recommended (beyond any factory; a failure turns
the feature off instead of holding the project). New required checks:
key switch rating, a fuse per drive motor, a locked-wheel heat test, a
10 degree slope hold, top speed for the rider's age, and edges. The 0.75 s
link-loss stop stays required.

The schematic gets F11-F14, a 15 A placeholder blade fuse in each drive
motor's + lead inside the box, so a single stalled motor has a hardware
backstop below the 20 A software limit and the 40 A main fuse. Variant B's
current sensors feed the same fuses. Safety review updated to match.
Parts:
- added F11, F12, F13, F14: 15 A, symbol Device:Fuse
Connections:
- net FL_M_POS: now also F11.2; no longer U10.M+
- net FR_M_POS: now also F12.2; no longer U11.M+
- net RL_M_POS: now also F13.2; no longer U12.M+
- net RR_M_POS: now also F14.2; no longer U13.M+
- new net FL_DRV_POS: F11.1, U10.M+
- new net FR_DRV_POS: F12.1, U11.M+
- new net RL_DRV_POS: F13.1, U12.M+
- new net RR_DRV_POS: F14.1, U13.M+
Other:
- note added: "F11-F14: a fuse in each drive motor's + lead, so a stalled wheel blows its own fuse (safety review M3)."
- moved on the sheet: C101, C102, C103, C104, C105, C111, C112, C113, C114, C115, D101, D102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
